File: PCB-demo.kicad_sch (KiCad schematic)
At the start: 0 parts

Commit message: Update gitignore
Other:
- company: (none) -> University of Virginia
- title: (none) -> PCB-demo
Changed lines of the file:
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@@
 	(generator "eeschema")
 	(generator_version "10.0")
-	(paper "A4")
+	(paper "USLedger")
+	(title_block
+		(title "PCB-demo")
+		(date "2026-09-24")
+		(rev "V0.9")
+		(company "University of Virginia")
+		(comment 1 "School of Engineering and Applied Sciences")
+		(comment 2 "Department of Mechanical and Aerospace Engineering")
+		(comment 3 "Mike McPherson")
+	)
 	(sheet_instances
 		(path "/"

Commit message: Complete schematic entry
Parts:
- added A1: RaspberryPi_Pico_W, Module:RaspberryPi_Pico_W_SMD_HandSolder, symbol MCU_Module:RaspberryPi_Pico_W
- added C1: 4u7, Capacitor_SMD:C_0603_1608Metric, symbol Device:C_Small
- added C2: 100u, Capacitor_SMD:C_0603_1608Metric, symbol Device:C_Polarized_Small_US
- added C3: 10u, Capacitor_SMD:C_0603_1608Metric, symbol Device:C_Small
- added C4, C6: 100n, Capacitor_SMD:C_0603_1608Metric, symbol Device:C_Small
- added C5: 2u2, Capacitor_SMD:C_0603_1608Metric, symbol Device:C_Small
- added C7: 22u, Capacitor_SMD:C_0603_1608Metric, symbol Device:C_Small
- added C8: 100n, Capacitor_SMD:CP_Elec_10x10, symbol Device:C_Small
- added D1: LED RED, LED_SMD:LED_0603_1608Metric, symbol Device:LED
- added J1: 22053021, Molex-22053021:CONN_A-7478-02A_MOL, symbol Molex-22053021:22053021
- added L1: 470n, Inductor_SMD:L_0603_1608Metric, symbol Device:L_Small
- added L2: 100u, Inductor_SMD:L_12x12mm_H6mm, symbol Device:L_Small
- added Q1: DMG2305UX-13, DMG2305UX_13:SOT91P240X110-3N, symbol DMG2305UX-13:DMG2305UX-13
- added R1: 0.1, Resistor_SMD:R_0603_1608Metric, symbol Device:R_Small_US
- added R2: 1k8, Resistor_SMD:R_0603_1608Metric, symbol Device:R_Small_US
- added U1: TPS543320RPYR, TPS543320RPYR:RPY0014A-MFG, symbol TPS543320RPYR:TPS543320RPYR
Connections:
- new net: C5.1, U1.6 (BP5)
- new net: C3.1, C4.1, L1.2, R1.1, U1.12 (VIN), U1.8 (VIN)
- new net: D1.1 (K), R2.1
- new net: A1.26 (GPIO20), D1.2 (A)
- new net: C1.1, J1.1, L1.1
- new net: C2.1, R1.2
- new net: C6.1, U1.14 (BOOT)
- new net: C6.2, L2.1, U1.10 (SW), U1.13 (SW)
- new net +5V: C7.1, C8.1, L2.2, Q1.3, U1.4 (FB)
- new net GND: A1.13 (GND), A1.18 (GND), A1.23 (GND), A1.28 (GND), A1.3 (GND), A1.33 (AGND), A1.38 (GND), A1.8 (GND), C1.2, C2.2, C3.2, C4.2, C5.2, C7.2, C8.2, J1.2, R2.2, U1.11 (PGND), U1.5 (AGND), U1.9 (PGND)
- new net VBUS: A1.40 (VBUS), Q1.1
- new net VSYS: A1.39 (VSYS), Q1.2
- no-connect marks 0 -> 33
